Commit message: Introduce experimental simulated multi-ranger deck
Built with four hokuyo sensors
For further information see:
https://github.com/Hokuyo-aut/urg_node2
https://github.com/ros-simulation/gazebo_ros_pkgs/wiki/ROS-2-Migration:-Ray-sensors

File: models/rotors_description/urdf/component_snippets.xacro (robot description, xacro)
@@ -190,4 +190,16 @@
     </gazebo>
   </xacro:macro>
+  <!-- Macro to add the mr_plugin. -->
+  <xacro:if value="${enable_mr_deck}">
+    <xacro:macro name="mr_plugin_macro" params="namespace rate">
+      <gazebo>
+        <plugin name="mr_plugin" filename="librotors_gazebo_mr_plugin.so">
+          <robotNamespace>${namespace}</robotNamespace>
+          <rate>${rate}</rate>
+          <visualize_ray>${mr_deck_visualize}</visualize_ray>
+        </plugin>
+      </gazebo>
+    </xacro:macro>
+  </xacro:if>
   <!-- Macro to add a generic odometry sensor. -->
   <xacro:macro name="odometry_plugin_macro"

File: models/rotors_description/urdf/crazyflie.xacro (robot description, xacro)
@@ -32,4 +32,33 @@
   <xacro:property name="rotor_drag_coefficient" value="9.1785e-7" />
   <xacro:property name="rolling_moment_coefficient" value="0.0000001" />
+  <!-- Multi-ranger deck -->
+  <xacro:property name="expansion_deck_offset" value="0.018" />
+  <xacro:property name="mr_deck_width" value="0.025" />
+  <xacro:property name="mr_deck_length" value="0.025" />
+  <xacro:property name="mr_deck_height" value="0.002" />
+  <xacro:property name="mr_deck_color" value="Black" />
+  <xacro:property name="sensor_box_offset" value="0.002" />
+  <xacro:property name="sensor_offset" value="0.005" />
+  <xacro:property name="sensor_box_yaw_front" value="0.0" />
+  <xacro:property name="sensor_box_yaw_back" value="3.14159" />
+  <xacro:property name="sensor_box_yaw_left" value="1.5708" />
+  <xacro:property name="sensor_box_yaw_right" value="-1.5708" />
+  <xacro:property name="mr_sensor_length" value="0.001" />
+  <xacro:property name="mr_sensor_width" value="0.01" />
+  <xacro:property name="mr_sensor_height" value="0.005" />
+  <xacro:property name="mr_sensor_trans_x_front" value="0.01" />
+  <xacro:property name="mr_sensor_trans_y_front" value="0.0" />
+  <xacro:property name="mr_sensor_trans_x_back" value="-0.01" />
+  <xacro:property name="mr_sensor_trans_y_back" value="0.0" />
+  <xacro:property name="mr_sensor_trans_x_left" value="0.0" />
+  <xacro:property name="mr_sensor_trans_y_left" value="0.01" />
+  <xacro:property name="mr_sensor_trans_x_right" value="0.0" />
+  <xacro:property name="mr_sensor_trans_y_right" value="-0.01" />
+  <xacro:property name="mr_sensor_color_front" value="Red" />
+  <xacro:property name="mr_sensor_color_back" value="Blue" />
+  <xacro:property name="mr_sensor_color_left" value="Green" />
+  <xacro:property name="mr_sensor_color_right" value="Yellow" />
+  <xacro:property name="mr_sensor_color_right" value="Yellow" />
+  <xacro:property name="mr_deck_visualize" value="$(arg mr_deck_visualize)" />
   <!-- Property Blocks -->
   <xacro:property name="body_inertia">
@@ -144,3 +173,67 @@
     <xacro:insert_block name="rotor_inertia" />
   </xacro:vertical_rotor>
+  <!-- Instantiate multi-ranger deck consisting
+       of a plane and four range sensors -->
+  <xacro:if value="${enable_mr_deck}">
+  <xacro:multiranger_deck_base
+    robot_namespace="${namespace}"
+    expansion_deck_offset="${expansion_deck_offset}"
+    mr_deck_width="${mr_deck_width}"
+    mr_deck_length="${mr_deck_length}"
+    mr_deck_height="${mr_deck_height}"
+    mr_deck_color="${mr_deck_color}">
+  </xacro:multiranger_deck_base>
+  <xacro:mr_range_sensor robot_namespace="${namespace}"
+    sensor_location="front"
+    sensor_box_offset="${sensor_box_offset}"
+    sensor_box_yaw="${sensor_box_yaw_front}"
+    trans_x="${mr_sensor_trans_x_front}"
+    trans_y="${mr_sensor_trans_y_front}"
+    sensor_length="${mr_sensor_length}"
+    sensor_width="${mr_sensor_width}"
+    sensor_height="${mr_sensor_height}"
+    sensor_offset="${sensor_offset}"
+    mr_sensor_color="${mr_sensor_color_front}"
+    visualize_ray="${mr_deck_visualize}">
+  </xacro:mr_range_sensor>
+  <xacro:mr_range_sensor robot_namespace="${namespace}"
+    sensor_location="back"
+    sensor_box_offset="${sensor_box_offset}"
+    sensor_box_yaw="${sensor_box_yaw_back}"
+    trans_x="${mr_sensor_trans_x_back}"
+    trans_y="${mr_sensor_trans_y_back}"
+    sensor_length="${mr_sensor_length}"
+    sensor_width="${mr_sensor_width}"
+    sensor_height="${mr_sensor_height}"
+    sensor_offset="${sensor_offset}"
+    mr_sensor_color="${mr_sensor_color_back}"
+    visualize_ray="${mr_deck_visualize}">
+  </xacro:mr_range_sensor>
+  <xacro:mr_range_sensor robot_namespace="${namespace}"
+    sensor_location="left"
+    sensor_box_offset="${sensor_box_offset}"
+    sensor_box_yaw="${sensor_box_yaw_left}"
+    trans_x="${mr_sensor_trans_x_left}"
+    trans_y="${mr_sensor_trans_y_left}"
+    sensor_length="${mr_sensor_length}"
+    sensor_width="${mr_sensor_width}"
+    sensor_height="${mr_sensor_height}"
+    sensor_offset="${sensor_offset}"
+    mr_sensor_color="${mr_sensor_color_left}"
+    visualize_ray="${mr_deck_visualize}">
+  </xacro:mr_range_sensor>
+  <xacro:mr_range_sensor robot_namespace="${namespace}"
+    sensor_location="right"
+    sensor_box_offset="${sensor_box_offset}"
+    sensor_box_yaw="${sensor_box_yaw_right}"
+    trans_x="${mr_sensor_trans_x_right}"
+    trans_y="${mr_sensor_trans_y_right}"
+    sensor_length="${mr_sensor_length}"
+    sensor_width="${mr_sensor_width}"
+    sensor_height="${mr_sensor_height}"
+    sensor_offset="${sensor_offset}"
+    mr_sensor_color="${mr_sensor_color_right}"
+    visualize_ray="${mr_deck_visualize}">
+  </xacro:mr_range_sensor>
+  </xacro:if>
 </robot>

File: models/rotors_description/urdf/crazyflie_base.xacro (robot description, xacro)
@@ -13,4 +13,5 @@
   <xacro:arg name='allow_collision' default='true' />
   <xacro:property name="enable_ground_truth" value="$(arg enable_ground_truth)" />
+  <xacro:property name="enable_mr_deck" value="$(arg enable_mr_deck)" />
   <xacro:include filename="$(arg rotors_description_dir)/urdf/component_snippets.xacro"/>
   <!-- Instantiate crazyflie "mechanics" -->
@@ -85,4 +86,10 @@
     rate="100">
   </xacro:lps_plugin_macro>
+  <xacro:if value="${enable_mr_deck}">
+    <xacro:mr_plugin_macro
+      namespace="${namespace}"
+      rate="100">
+    </xacro:mr_plugin_macro>
+  </xacro:if>
   <xacro:if value="${enable_ground_truth}">
     <!-- Odometry Sensor -->

File: models/rotors_description/urdf/multirotor_base.xacro (robot description, xacro)
@@ -143,3 +143,89 @@
     </gazebo>
   </xacro:macro>
+    <!-- Multi-ranger deck plane -->
+  <xacro:macro name="multiranger_deck_base" params="robot_namespace expansion_deck_offset mr_deck_width mr_deck_length mr_deck_height mr_deck_color">
+    <joint name="base_mr_joint" type="fixed">
+      <origin xyz="0 0 ${expansion_deck_offset}" rpy="0 0 0" />
+      <parent link="base_link"/>
+      <child link="multi_ranger_deck_plane_link"/>
+    </joint>
+    <link name="multi_ranger_deck_plane_link">
+      <visual>
+        <origin xyz="0 0 0" rpy="0 0 0" />
+        <geometry>
+          <box size="${mr_deck_width} ${mr_deck_length} ${mr_deck_height}"/>
+        </geometry>
+      </visual>
+    </link>
+    <gazebo reference="multi_ranger_deck_plane_link">
+      <material>Gazebo/${mr_deck_color}</material>
+    </gazebo>
+  </xacro:macro>
+  <!-- Multi-ranger range sensor -->
+  <!-- https://github.com/ros-simulation/gazebo_ros_pkgs/wiki/ROS-2-Migration:-Ray-sensors -->
+  <xacro:macro name="mr_range_sensor" params="robot_namespace sensor_location sensor_box_offset sensor_box_yaw trans_x trans_y sensor_length sensor_width sensor_height sensor_offset mr_sensor_color visualize_ray">
+    <joint name="mr_sensor_${sensor_location}_joint" type="fixed">
+      <!-- <origin xyz="${trans_x} ${trans_y} ${sensor_box_offset}+${sensor_offset}" rpy="0 0 ${sensor_box_yaw}" /> -->
+      <origin xyz="${trans_x} ${trans_y} ${sensor_box_offset}" rpy="0 0 ${sensor_box_yaw}" />
+      <parent link="multi_ranger_deck_plane_link"/>
+      <child link="mr_sensor_${sensor_location}_link"/>
+    </joint>
+    <link name="mr_sensor_${sensor_location}_link">
+      <!-- To avoid that the sensor interferes with the link we disable the collision -->
+      <!-- <collision>
+        <origin xyz="0 0 0" rpy="0 0 0"/>
+        <geometry>
+          <box size="${sensor_length} ${sensor_width} ${sensor_height}"/>
+        </geometry>
+      </collision> -->
+      <visual>
+        <origin xyz="0 0 0" rpy="0 0 0" />
+        <geometry>
+          <box size="${sensor_length} ${sensor_width} ${sensor_height}"/>
+        </geometry>
+      </visual>
+    </link>
+    <gazebo reference="mr_sensor_${sensor_location}_link">
+      <material>Gazebo/${mr_sensor_color}</material>
+    </gazebo>
+    <gazebo reference="mr_sensor_${sensor_location}_link">
+      <sensor type="ray" name="head_hokuyo_sensor_${sensor_location}">
+          <pose>0 0 0 0 0 0</pose>
+          <visualize>${visualize_ray}</visualize>
+          <ray>
+            <scan>
+                <horizontal>
+                  <samples>1</samples>
+                  <resolution>1.0</resolution>
+                  <min_angle>-0.01</min_angle>
+                  <max_angle>0.01</max_angle>
+                </horizontal>
+                <vertical>
+                  <samples>1</samples>
+                  <resolution>1</resolution>
+                  <min_angle>-0.01</min_angle>
+                  <max_angle>0.01</max_angle>
+                </vertical>
+            </scan>
+            <range>
+                <min>0.05</min>
+                <max>4.00</max>
+                <resolution>0.02</resolution>
+            </range>
+          </ray>
+          <update_rate>15</update_rate>
+          <plugin filename="libgazebo_ros_ray_sensor.so" name="gazebo_ros_range_${namespace}_${sensor_location}">
+            <ros>
+              <namespace>/${namespace}/${sensor_location}</namespace>
+              <remapping>~/out:=range</remapping>
+            </ros>
+            <output_type>sensor_msgs/Range</output_type>
+            <gaussianNoise>0.005</gaussianNoise>
+            <radiation_type>infrared</radiation_type>
+            <alwaysOn>true</alwaysOn>
+            <fov>0.02</fov>
+          </plugin>
+      </sensor>
+    </gazebo>
+  </xacro:macro>
 </robot>

Commit message: Implement TDoA plugin

File: models/rotors_description/urdf/component_snippets.xacro (robot description, xacro)
@@ -202,4 +202,12 @@
     </xacro:macro>
   </xacro:if>
+  <!-- Macro to add the tdoa_plugin. -->
+  <xacro:macro name="tdoa_plugin_macro" params="namespace">
+    <gazebo>
+      <plugin name="tdoa_plugin" filename="librotors_gazebo_tdoa_plugin.so">
+        <robotNamespace>${namespace}</robotNamespace>
+      </plugin>
+    </gazebo>
+  </xacro:macro>
   <!-- Macro to add a generic odometry sensor. -->
   <xacro:macro name="odometry_plugin_macro"

File: models/rotors_description/urdf/crazyflie_base.xacro (robot description, xacro)
@@ -92,4 +92,7 @@
     </xacro:mr_plugin_macro>
   </xacro:if>
+  <xacro:tdoa_plugin_macro
+    namespace="${namespace}">
+  </xacro:tdoa_plugin_macro>
   <xacro:if value="${enable_ground_truth}">
     <!-- Odometry Sensor -->
